File: IkeaTradfriLEDdriver.kicad_pcb (KiCad board)
At the start: 2 copper layers, 74.9 x 43.2 mm, 9 parts, among them J1 Conn_01x02_Male, J2 Conn_01x02_Male, J3 Conn_01x02_Male, Q1 BUZ11, U1 LM741

Commit message: pokusy na desce
Parts:
- J1: value Conn_01x02_Male -> input
- J2: value Conn_01x02_Male -> PWM
- J3: value Conn_01x02_Male -> LED strip
- moved J2 44.9 mm to (138.4, 39.4)
- moved R1 26.7 mm to (137.7, 49.8), turned to 0 degrees
- moved J3 15.3 mm to (193.0, 54.6), turned to 270 degrees
- moved J1 12.5 mm to (127.0, 55.9)
- moved D1 12.0 mm to (137.7, 45.2), turned to 0 degrees
- moved R3 11.4 mm to (160.0, 50.8), turned to 270 degrees
- moved R2 8.64 mm to (132.7, 44.5), turned to 270 degrees
- moved Q1 5.24 mm to (167.6, 54.6)
Connections:
- R1 pad 1: +12V -> Net-(D1-Pad1)
- R1 pad 2: Net-(D1-Pad1) -> +12V
- U1 pad 1: Net-(U1-Pad1) -> (no net)
- U1 pad 3: Net-(U1-Pad3) -> Net-(D1-Pad1)
- U1 pad 5: Net-(U1-Pad5) -> (no net)
- U1 pad 8: Net-(U1-Pad8) -> (no net)
Routing:
- net GND: track 113.0 -> 0.00 mm, vias 5 -> 0
- net Net-(J2-Pad1): track 54.9 -> 10.1 mm
- net +12V: track 64.5 -> 39.5 mm
- net Net-(R3-Pad2): track 0.00 -> 6.88 mm
- net Net-(R3-Pad1): track 6.35 -> 0.00 mm
- net Net-(Q1-Pad1): track 15.8 -> 9.59 mm
- net Net-(D1-Pad1): track 46.6 -> 52.5 mm
- net Net-(J3-Pad1): track 31.8 -> 26.5 mm
- net Net-(R2-Pad2): track 15.3 -> 11.8 mm
- removed copper zone on F.Cu, net GND
